File: TIA_mplifier.kicad_pcb (KiCad board)
At the start: 2 copper layers, 76.7 x 46.3 mm, 22 parts, among them J1 RF_in, J2 Screw_Terminal_01x02, J3 RF_out, Q1 2N3904, Q2 2N3904, Q3 2N3904

Commit message: added production zip file
Connections:
- JP1 pad : GND -> (no net)
Routing:
- net Net-(Q2-C): track 90.3 -> 95.6 mm
- net Net-(Q1-C): track 45.4 -> 50.2 mm
